File: 486 Breakout.sch (KiCad schematic (older format))
At the start: 37 parts, among them J1 PWR, J10 Conn_02x03_Counter_Clockwise, J11 Cache FPU, J12 Parity, J13 Bus Size Byte Enabled, J14 Bus Arbitration, J2 Not Connected, J3 Address Bus, J4 Data Bus, J5 CLK, J6 Conn_02x03_Counter_Clockwise, J7 Int, J8 Control Bus, J9 Conn_02x04_Counter_Clockwise, SW1 POWER, SW2 RESET

Commit message: V2 of the board
Parts:
- removed J7: Int, Connector_PinHeader_2.54mm:PinHeader_1x02_P2.54mm_Vertical, symbol Connector:Conn_01x02_Male
- removed R20: 10k, Resistor_THT:R_Axial_DIN0204_L3.6mm_D1.6mm_P5.08mm_Horizontal, symbol Device:R
- removed SW1: POWER, Button_Switch_THT:SW_NKK_G1xJP, symbol Switch:SW_DPDT_x2
- removed SW2: RESET, Button_Switch_THT:SW_PUSH_6mm_H5mm, symbol Switch:SW_Push
- added J12: FPU, Connector_PinHeader_2.54mm:PinHeader_1x02_P2.54mm_Vertical, symbol Connector:Conn_01x02_Male
- added J14: Bus Size, Connector_PinHeader_2.54mm:PinHeader_1x02_P2.54mm_Vertical, symbol Connector:Conn_01x02_Male
- added R14: 10k, Resistor_THT:R_Axial_DIN0204_L3.6mm_D1.6mm_P7.62mm_Horizontal, symbol Device:R
- D1: value LED_ALT -> POWER
- J11: renamed from J13; value Bus Size Byte Enabled -> Byte Enabled; footprint Connector_PinHeader_2.54mm:PinHeader_1x08_P2.54mm_Vertical -> Connector_PinHeader_2.54mm:PinHeader_1x06_P2.54mm_Vertical; symbol Connector:Conn_01x08_Male -> Connector:Conn_01x06_Male
- J13: renamed from J5; value CLK -> Input; footprint Connector_PinHeader_2.54mm:PinHeader_1x01_P2.54mm_Vertical -> Connector_PinHeader_2.54mm:PinHeader_1x04_P2.54mm_Vertical; symbol Connector:Conn_01x01_Male -> Connector:Conn_01x04_Male
- J7: renamed from J8; footprint Connector_PinHeader_2.54mm:PinHeader_1x10_P2.54mm_Vertical -> Connector_PinHeader_2.54mm:PinHeader_1x09_P2.54mm_Vertical; symbol Connector:Conn_01x10_Male -> Connector:Conn_01x09_Male
- J8: renamed from J11; value Cache FPU -> Cache; footprint Connector_PinHeader_2.54mm:PinHeader_1x08_P2.54mm_Vertical -> Connector_PinHeader_2.54mm:PinHeader_1x06_P2.54mm_Vertical; symbol Connector:Conn_01x08_Male -> Connector:Conn_01x06_Male
- R1: footprint Resistor_THT:R_Axial_DIN0204_L3.6mm_D1.6mm_P5.08mm_Horizontal -> Resistor_THT:R_Axial_DIN0204_L3.6mm_D1.6mm_P7.62mm_Horizontal
- R10: renamed from R12; footprint Resistor_THT:R_Axial_DIN0204_L3.6mm_D1.6mm_P5.08mm_Horizontal -> Resistor_THT:R_Axial_DIN0204_L3.6mm_D1.6mm_P7.62mm_Horizontal
- R11: renamed from R13; footprint Resistor_THT:R_Axial_DIN0204_L3.6mm_D1.6mm_P5.08mm_Horizontal -> Resistor_THT:R_Axial_DIN0204_L3.6mm_D1.6mm_P7.62mm_Horizontal
- R12: renamed from R14; footprint Resistor_THT:R_Axial_DIN0204_L3.6mm_D1.6mm_P5.08mm_Horizontal -> Resistor_THT:R_Axial_DIN0204_L3.6mm_D1.6mm_P7.62mm_Horizontal
- R13: renamed from R15; footprint Resistor_THT:R_Axial_DIN0204_L3.6mm_D1.6mm_P5.08mm_Horizontal -> Resistor_THT:R_Axial_DIN0204_L3.6mm_D1.6mm_P7.62mm_Horizontal
- R15: renamed from R16; footprint Resistor_THT:R_Axial_DIN0204_L3.6mm_D1.6mm_P5.08mm_Horizontal -> Resistor_THT:R_Axial_DIN0204_L3.6mm_D1.6mm_P7.62mm_Horizontal
- R16: renamed from R17; footprint Resistor_THT:R_Axial_DIN0204_L3.6mm_D1.6mm_P5.08mm_Horizontal -> Resistor_THT:R_Axial_DIN0204_L3.6mm_D1.6mm_P7.62mm_Horizontal
- R17: renamed from R18; footprint Resistor_THT:R_Axial_DIN0204_L3.6mm_D1.6mm_P5.08mm_Horizontal -> Resistor_THT:R_Axial_DIN0204_L3.6mm_D1.6mm_P7.62mm_Horizontal
- R18: renamed from R19; footprint Resistor_THT:R_Axial_DIN0204_L3.6mm_D1.6mm_P5.08mm_Horizontal -> Resistor_THT:R_Axial_DIN0204_L3.6mm_D1.6mm_P7.62mm_Horizontal
- R19: renamed from R2; footprint Resistor_THT:R_Axial_DIN0204_L3.6mm_D1.6mm_P5.08mm_Horizontal -> Resistor_THT:R_Axial_DIN0204_L3.6mm_D1.6mm_P7.62mm_Horizontal
- R2: renamed from R4; footprint Resistor_THT:R_Axial_DIN0204_L3.6mm_D1.6mm_P5.08mm_Horizontal -> Resistor_THT:R_Axial_DIN0204_L3.6mm_D1.6mm_P7.62mm_Horizontal
- R20: renamed from R3; footprint Resistor_THT:R_Axial_DIN0204_L3.6mm_D1.6mm_P5.08mm_Horizontal -> Resistor_THT:R_Axial_DIN0204_L3.6mm_D1.6mm_P7.62mm_Horizontal
- R3: renamed from R5; footprint Resistor_THT:R_Axial_DIN0204_L3.6mm_D1.6mm_P5.08mm_Horizontal -> Resistor_THT:R_Axial_DIN0204_L3.6mm_D1.6mm_P7.62mm_Horizontal
- R4: renamed from R6; footprint Resistor_THT:R_Axial_DIN0204_L3.6mm_D1.6mm_P5.08mm_Horizontal -> Resistor_THT:R_Axial_DIN0204_L3.6mm_D1.6mm_P7.62mm_Horizontal
- R5: renamed from R7; footprint Resistor_THT:R_Axial_DIN0204_L3.6mm_D1.6mm_P5.08mm_Horizontal -> Resistor_THT:R_Axial_DIN0204_L3.6mm_D1.6mm_P7.62mm_Horizontal
- R6: renamed from R8; footprint Resistor_THT:R_Axial_DIN0204_L3.6mm_D1.6mm_P5.08mm_Horizontal -> Resistor_THT:R_Axial_DIN0204_L3.6mm_D1.6mm_P7.62mm_Horizontal
- R7: renamed from R9; footprint Resistor_THT:R_Axial_DIN0204_L3.6mm_D1.6mm_P5.08mm_Horizontal -> Resistor_THT:R_Axial_DIN0204_L3.6mm_D1.6mm_P7.62mm_Horizontal
- R8: renamed from R10; footprint Resistor_THT:R_Axial_DIN0204_L3.6mm_D1.6mm_P5.08mm_Horizontal -> Resistor_THT:R_Axial_DIN0204_L3.6mm_D1.6mm_P7.62mm_Horizontal
- R9: renamed from R11; footprint Resistor_THT:R_Axial_DIN0204_L3.6mm_D1.6mm_P5.08mm_Horizontal -> Resistor_THT:R_Axial_DIN0204_L3.6mm_D1.6mm_P7.62mm_Horizontal
- renumbered J14 to J15, J9 to J2, J2 to J3, J3 to J4, J4 to J5, J12 to J9
Connections:
- net +5V: now also J1.1 (Pin_1)
- net GND: now also R14.2
- net INTR: now also J13.3 (Pin_3), R17.1; no longer R18.1
- net NMI: now also J13.4 (Pin_4), R18.1; no longer R17.1
- net PCD: now also J12.2 (Pin_2); no longer J8.8 (Pin_8)
- net PWT: now also J12.1 (Pin_1); no longer J8.7 (Pin_7)
- net RESET: now also J13.2 (Pin_2), R14.1; no longer J7.10 (Pin_10)
- net at R7.1: now also J2.8 (Pin_8); no longer J2.2 (Pin_2)
- net at R6.1: now also J2.6 (Pin_6); no longer J2.4 (Pin_4)
- net at R5.1: now also J2.4 (Pin_4); no longer J2.6 (Pin_6)
- net at R4.1: now also J2.2 (Pin_2); no longer J2.8 (Pin_8)
- net A20M* renamed A20M#
- net A20M#: now also R2.1; no longer R3.1
- net ADS* renamed ADS#
- net BE0* renamed BE0#
- net BE1* renamed BE1#
- net BE2* renamed BE2#
- net BE3* renamed BE3#
- net BLAST* renamed BLAST#
- net BOFF* renamed BOFF#
- net BRDY* renamed BRDY#
- net BRDY#: now also R20.1; no longer R20.2
- net BRDY*R renamed BRDY#R
- net BRDY#R: now also R20.2; no longer R20.1
- net BS16* renamed BS8#
- net BS8#: now also J14.1 (Pin_1); no longer J11.8 (Pin_8)
- net BS8* renamed BS16#
- net BS16#: now also J14.2 (Pin_2); no longer J11.7 (Pin_7)
- net D_C* renamed D_C#
- net EADS* renamed EADS#
- net FERR* renamed FERR#
- net FLUSH* renamed FLUSH#
- net IGNNE* renamed IGNNE#
- net IGNNE#: now also R3.1; no longer R9.1
- net KEN* renamed KEN#
- net KEN#: now also R9.1; no longer R2.1
- net LOCK* renamed LOCK#
- net M_IO* renamed M_IO#
- net PCHK* renamed PCHK#
- net PLOCK* renamed PLOCK#
- net RDY* renamed RDY#
- net RDY*R renamed RDY#R
- net W_R* renamed W_R#
- no-connect marks 1 -> 0
Other:
- moved on the sheet: D1, J1, J10, J15, J2, J9, R1, R10, R11, R12, R13, R15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
