File: CPUSheet.sch (KiCad schematic (older format))
At the start: 13 parts, among them U1 80486, U2 7400, U3 7400

Commit message: V2 of the board
Parts:
- C1, C10, C2, C3, C4, C5, C6, C7, C8, C9: value C -> 105
- U1: value 80486 -> 80486DX
Connections:
- net A20M* renamed A20M#
- net ADS* renamed ADS#
- net BE0* renamed BE0#
- net BE1* renamed BE1#
- net BE2* renamed BE2#
- net BE3* renamed BE3#
- net BLAST* renamed BLAST#
- net BOFF* renamed BOFF#
- net BRDY* renamed BRDY#
- net BS16* renamed BS16#
- net BS8* renamed BS8#
- net D_C* renamed D_C#
- net EADS* renamed EADS#
- net FERR* renamed FERR#
- net FLUSH* renamed FLUSH#
- net IGNNE* renamed IGNNE#
- net KEN* renamed KEN#
- net LOCK* renamed LOCK#
- net M_IO* renamed M_IO#
- net PCHK* renamed PCHK#
- net PLOCK* renamed PLOCK#
- net RDY* renamed RDY#
- net W_R* renamed W_R#
Other:
- note added: "A1, BHE#, BLE# Logic Provided by the 486 Data Sheet"
- note added: "BLE# is also A0"
